File: KiCAD/1.0/uproszczony_odbiornik.kicad_sch (KiCad schematic)
At the start: 55 parts, among them IC4 DSPIC33FJ64MC804-PT, Q1 10MHz, Y1 CMR309T

Commit message: fix schematics and PCB, Add R2
Parts:
- added R2: 20k, uproszczony_odbiornik:R0805, symbol uproszczony_odbiornik-eagle-import:R-EU_R0805
Connections:
- net VDD: now also R2.2
- net at IC4.23 (AN4/C1IN-/RP2/CN6/RB2), SV2.3: now also R2.1
Other:
- note added: "Złącze Wyświetlacza"
- note added: "konsola szeregowa"
- moved on the sheet: ANT0, C1, C10, C12, C13, C14, C15, C17, C18, C19, C2, C21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
